File: Hardware/MSP430_G2_PDIP20_Devboard_THT/MSP430_G2_PDIP20_Devboard_THT.kicad_sch (KiCad schematic)
At the start: 0 parts

Commit message: MSP430 G2 PDIP20 Dev Board - Schematics - Placed Components
Signed-off-by: alexanderjg85 <alexanderjg85@gmail.com>
Parts:
- added C1, C2: 1 uF, AJ_Passives:C6119929_C0805, symbol Device:C_Small
- added C3: 1 nF, AJ_Passives:C141155_C0805, symbol AJ_Passives:C0805F102K1RACAUTO
- added C5: 100nF, AJ_Passives:C49678_C0805, symbol Device:C_Small
- added D1: SS14, Diode_SMD:D_SMA_Handsoldering, symbol Diode:SS14
- added D2: GREEN, LED_THT:LED_D3.0mm, symbol Device:LED
- added D3: YELLOW, LED_THT:LED_D3.0mm, symbol Device:LED
- added J1: 2479774-1, AJ_Connectors:24797741, symbol AJ_Connectors:2479774-1
- added J2: Conn_01x04_Pin, Connector_PinHeader_2.54mm:PinHeader_1x04_P2.54mm_Vertical, symbol Connector:Conn_01x04_Pin
- added J3: Conn_01x10_Pin, Connector_PinHeader_2.54mm:PinHeader_1x10_P2.54mm_Vertical, symbol Connector:Conn_01x10_Pin
- added J4: Conn_01x10_Pin, symbol Connector:Conn_01x10_Pin
- added JP1: JP_PLED, TestPoint:TestPoint_2Pads_Pitch2.54mm_Drill0.8mm, symbol Jumper:Jumper_2_Small_Open
- added JP3: JP_SLED, TestPoint:TestPoint_2Pads_Pitch2.54mm_Drill0.8mm, symbol Jumper:Jumper_2_Small_Open
- added R1: 470, Resistor_SMD:R_1206_3216Metric_Pad1.30x1.75mm_HandSolder, symbol Device:R_Small
- added R2: 47k, Resistor_SMD:R_1206_3216Metric_Pad1.30x1.75mm_HandSolder, symbol Device:R_Small
- added R3: 330, Resistor_SMD:R_1206_3216Metric_Pad1.30x1.75mm_HandSolder, symbol Device:R_Small
- added R4, R5: R_Small, symbol Device:R_Small
- added R6, R7: FRC0805F5101TS, AJ_Passives:C2907269_R0805, symbol AJ_Passives:FRC0805F5101TS
- added SW1: SW_RESET, AJ_Electromechanical:SW_SPST_PTS647_Sx38_Handsolder, symbol Switch:SW_Push
- added TP2: SLED, TestPoint:TestPoint_Pad_D1.5mm, symbol Connector:TestPoint
- added U1: MSP430G2302IN20, Package_DIP:DIP-20_W7.62mm, symbol MCU_Texas_MSP430:MSP430G2302IN20
- added U2: AP2112K-3.3TRG1(MS), AJ_Power:C22365427_SOT-23-5_L2_9-W1_6-P0_95-LS2_7-BR, symbol AJ_Power:AP2112K-3_3TRG1(MS)
- added U3: PESD5V0S1BA_C5261083, AJ_Passives:C5261083_SOD-323_L1_7-W1_3-LS2_5-BI, symbol AJ_Passives:PESD5V0S1BA_C5261083
Connections:
- new net: D2.2 (A), R1.2
- new net: JP3.2 (B), R1.1, TP2.1
- new net: R4.2, R5.1, U2.3 (EN)
- new net: JP1.1 (A), R3.1
- new net: D3.2 (A), R3.2
- new net GND: C3.2, D2.1 (K), D3.1 (K), SW1.2
- new net MSP_LED: JP3.1 (A)
- new net MSP_RST: C3.1, R2.2, SW1.1
- new net VDD: JP1.2 (B), R2.1

Commit message: MSP430 G2 PDIP20 Dev Board - Schematics - Wired Power related signals and components
Signed-off-by: alexanderjg85 <alexanderjg85@gmail.com>
Parts:
- R4: value R_Small -> 33k; footprint (none) -> Resistor_SMD:R_0805_2012Metric_Pad1.20x1.40mm_HandSolder
- R5: value R_Small -> 100k; footprint (none) -> Resistor_SMD:R_0805_2012Metric_Pad1.20x1.40mm_HandSolder; LCSC (none) -> C17407
- R6, R7: value FRC0805F5101TS -> 5k1; symbol AJ_Passives:FRC0805F5101TS -> Device:R_Small
Connections:
- net GND: now also C1.2, C2.2, C5.2, J1.1 (MH1), J1.2 (MH2), J1.3 (MH3), J1.4 (MH4), J1.A12 (GND_1), J1.B12 (GND_2), R5.2, R6.2, R7.2, U1.20 (DVSS), U2.2 (GND), U3.2
- net VDD: now also C2.1, C5.1, D1.2 (A), U1.1 (DVCC), U2.5 (VOUT)
- net at R6.1: now also J1.A5 (CC1)
- net at R7.1: now also J1.B5 (CC2)
- net VCC: now reaches U3.1
- net VCC: now also C1.1, D1.1 (K), J1.A9 (VBUS_1), J1.B9 (VBUS_2), R4.1, U2.1 (VIN)
- no-connect marks 0 -> 1
Other:
- moved on the sheet: C1, C5, U3

Commit message: MSP430 G2 PDIP20 Dev Board - Schematics - Wirring finsished
Signed-off-by: alexanderjg85 <alexanderjg85@gmail.com>
Connections:
- net GND: now also J2.4 (Pin_4), J3.10 (Pin_10), J4.10 (Pin_10)
- net MSP_LED: now also J4.2 (Pin_2), U1.8 (P2.0)
- net MSP_RST: now also J2.2 (Pin_2), U1.16 (~{RST}/NMI/SBWTDIO)
- net VDD: now also J2.1 (Pin_1), J3.1 (Pin_1), J4.1 (Pin_1)
- net MSP_TEST: now reaches J2.3 (Pin_3)
- net MSP_TEST: now also U1.17 (SBWTCK/TEST)
- net P1.0: now reaches J3.2 (Pin_2)
- net P1.0: now also U1.2 (TA0CLK/ACLK/P1.0)
- net P1.1: now reaches J3.3 (Pin_3)
- net P1.1: now also U1.3 (TA0.0/P1.1)
- net P1.2: now reaches J3.4 (Pin_4)
- net P1.2: now also U1.4 (TA0.1/P1.2)
- net P1.3: now reaches J3.5 (Pin_5)
- net P1.3: now also U1.5 (P1.3)
- net P1.4: now reaches J3.6 (Pin_6)
- net P1.4: now also U1.6 (SMCLK/TCK/TA0.2/P1.4)
- net P1.5: now reaches J3.7 (Pin_7)
- net P1.5: now also U1.7 (TMS/TA0.0/P1.5)
- net P1.6: now reaches J3.8 (Pin_8)
- net P1.6: now also U1.14 (SDO/SCL/TDI/TCLK/TA0.1/P1.6)
- net P1.7: now reaches J3.9 (Pin_9)
- net P1.7: now also U1.15 (SDI/SDA/TDO/TDI/P1.7)
- net P2.1: now reaches J4.3 (Pin_3)
- net P2.1: now also U1.9 (P2.1)
- net P2.2: now reaches J4.4 (Pin_4)
- net P2.2: now also U1.10 (P2.2)
- net P2.3: now reaches J4.5 (Pin_5)
- net P2.3: now also U1.11 (P2.3)
- net P2.4: now reaches J4.6 (Pin_6)
- net P2.4: now also U1.12 (P2.4)
- net P2.5: now reaches J4.7 (Pin_7)
- net P2.5: now also U1.13 (P2.5)
- net P2.6: now reaches J4.8 (Pin_8)
- net P2.6: now also U1.19 (P2.6/XIN/TA0.1)
- net P2.7: now reaches J4.9 (Pin_9)
- net P2.7: now also U1.18 (P2.7/XOUT)
Other:
- moved on the sheet: J3, J4

Commit message: MSP430 G2 PDIP20 Dev Board - Schematics - Added Testpoints
Signed-off-by: alexanderjg85 <alexanderjg85@gmail.com>
Parts:
- added TP1: VDD, TestPoint:TestPoint_Pad_D1.5mm, symbol Connector:TestPoint
- added TP3: VCC, TestPoint:TestPoint_Pad_D1.5mm, symbol Connector:TestPoint
- added TP4, TP8: GND, TestPoint:TestPoint_Pad_D1.5mm, symbol Connector:TestPoint
- added TP5: EN, TestPoint:TestPoint_Pad_D1.5mm, symbol Connector:TestPoint
- added TP6: RES, TestPoint:TestPoint_Pad_D1.5mm, symbol Connector:TestPoint
- added TP7: TEST, TestPoint:TestPoint_Pad_D1.5mm, symbol Connector:TestPoint
Connections:
- net GND: now also TP4.1, TP8.1
- net MSP_RST: now also TP6.1
- net MSP_TEST: now also TP7.1
- net VCC: now also TP3.1
- net VDD: now also TP1.1
- net at R4.2, R5.1, U2.3 (EN): now also TP5.1

Commit message: MSP430 G2 PDIP20 Dev Board - Schematics - Assigned Footprint to Pinheader J4
Signed-off-by: alexanderjg85 <alexanderjg85@gmail.com>
Parts:
- J4: footprint (none) -> Connector_PinHeader_2.54mm:PinHeader_1x10_P2.54mm_Vertical
Changed lines of the file:
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@@
 			)
 		)
-		(property "Footprint" ""
+		(property "Footprint" "Connector_PinHeader_2.54mm:PinHeader_1x10_P2.54mm_Vertical"
 			(at 162.56 85.09 0)
 			(hide yes)

Commit message: MSP430 G2 PDIP20 Dev Board - Added BOM
Signed-off-by: alexanderjg85 <alexanderjg85@gmail.com>
Parts:
- C3: Package (none) -> 0805; Spec (none) -> ±10% 100V
- J1: Height 3.31 -> (none); MFR PN (none) -> 2479774-1; Manufacturer (none) -> TE Connectivity; Manufacturer_Name TE Connectivity -> (none); Manufacturer_Part_Number 2479774-1 -> (none); Mouser Part Number 571-2479774-1 -> (none); Mouser Price/Stock https://www.mouser.co.uk/ProductDetail/TE-Connectivity/2479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 -> (none); Package (none) -> Receptable 1x6; Spec (none) -> USB C 2.0
- J2: Package (none) -> 2.54 mm 1x4; Spec (none) -> Male / THT/ Vertical
- J3, J4: Package (none) -> 2.54 mm 1x10; Spec (none) -> Male / THT/ Vertical
- R4, R5, R6, R7: Package (none) -> 0805; Spec (none) -> 1% 125 mW
- U1: value MSP430G2302IN20 -> MSP430G2302; MFR PN (none) -> MSP430G2302IN20; Package (none) -> PDIP-20; Spec (none) -> 16-Bit MSP430 16 MHz
- U2: Package (none) -> SOT-23-5; Spec (none) -> 3V3 0.6 A
- U3: Package (none) -> SOD-323; Spec (none) -> Vbr 5.6V Vc 8V Ipp 11A
